File: ESP32-C3-WROOM_flexypin.kicad_pcb (KiCad board)
At the start: 2 copper layers, 31 x 28.6 mm, 25 parts, among them J1 Conn_01x09, J10 Conn_01x01, J11 Conn_01x01, J12 Conn_01x01, J13 Conn_01x01, J14 Conn_01x01, J15 Conn_01x01, J16 Conn_01x01, J17 Conn_01x01, J18 Conn_01x01, J2 Conn_01x01, J22 Conn_01x09, J23 Conn_01x01, J3 Conn_01x01, J4 Conn_01x01, J5 Conn_01x01, J6 Conn_01x01, J7 Conn_01x01, J8 Conn_01x01, J9 Conn_01x01

Commit message: made the C3
Parts:
- removed G*** (x2): LOGO, LOGO
- removed G*** (x2): LOGO, Symbols_Extra:SolderParty-New-Logo_5x4.2mm_SilkScreen
- removed J10, J11, J12, J13, J14, J15, J16, J17, J18, J23, J4, J5, J6, J7, J8, J9: Conn_01x01, FlexyPin:FlexyPin_1x01
- removed REF**: Fiducial_0.5mm_Mask1.5mm, Fiducial:Fiducial_0.5mm_Mask1.5mm
- added C1: 1µF, Capacitor_SMD:C_0402_1005Metric, F.Cu at (154.5, 96.1)
- added C2: 1µF, Capacitor_SMD:C_0402_1005Metric, F.Cu at (157.1, 97.9)
- added D1: D, Diode_SMD:D_SOD-323, F.Cu at (151.4, 98.4)
- added J19: USB_C_Receptacle_USB2.0_14P, Connector_USB:USB_C_Receptacle_G-Switch_GT-USB-7010ASV, F.Cu at (148.1, 105.7)
- added R1: 5,1kΩ, Resistor_SMD:R_0402_1005Metric, F.Cu at (149.8, 99.8)
- added R2: 5,1kΩ, Resistor_SMD:R_0402_1005Metric, F.Cu at (145.8, 100.3)
- added R3: 10kΩ, Resistor_SMD:R_0402_1005Metric, F.Cu at (155.6, 101.0)
- added SW1: SW_Push, Button_Switch_SMD:SW_Push_SPST_NO_Alps_SKRK, F.Cu at (141.0, 104.3)
- added SW3: SW_Push, Button_Switch_SMD:SW_Push_SPST_NO_Alps_SKRK, F.Cu at (155.1, 104.3)
- added U1: RT9080, Package_TO_SOT_SMD:SOT-23-5, F.Cu at (154.5, 98.3)
- J2, J3: value Conn_01x01 -> Conn_01x09; footprint FlexyPin:FlexyPin_1x01 -> flexypin:FlexyPin_1x09_P1.50mm
- moved J3 24.4 mm to (159.1, 93.3), turned to 180 degrees
Connections:
- net /3.3V renamed +3.3V
- J1 pad 2: /EN -> EN
- J1 pad 8: /IO9 -> IO9
- J1 pad 9: /GND -> GND
- J22 pad 5: /IO19 -> IO19
- J22 pad 6: /IO18 -> IO18
- J3 pad 1: /EN -> /IO10
Routing:
- net EN: track 0.00 -> 43.0 mm
- net IO19: track 0.00 -> 30.5 mm, vias 0 -> 2
- net IO18: track 0.00 -> 27.1 mm
- net IO9: track 0.00 -> 18.3 mm, vias 0 -> 1
- net +5V: track 0.00 -> 10.2 mm
- net GND: track 0.00 -> 10.0 mm
- net /GND: track 10.0 -> 0.00 mm
- net /IO9: track 9.66 -> 0.00 mm
- net /IO18: track 7.61 -> 0.00 mm
- net /IO19: track 6.68 -> 0.00 mm
- net Net-(D1-K): track 0.00 -> 6.25 mm
- net /EN: track 3.57 -> 0.00 mm
- net Net-(J19-CC1): track 0.00 -> 1.89 mm
- net Net-(J19-CC2): track 0.00 -> 1.68 mm
- net +3.3V: track 3.14 -> 3.34 mm, vias 0 -> 2
- added copper zone on B.Cu, net +3.3V
- added copper zone on F.Cu, net GND
Other:
- board text added: "BOOT"
- board text added: "RST"
- board text removed: "ESP32-C3-WROOM Adapter Jan 2022"
- board text removed: "Module on this side"
