File: ESP32-C3-WROOM_flexypin.kicad_sch (KiCad schematic)
At the start: 20 parts, among them J1 Conn_01x09, J10 Conn_01x01, J11 Conn_01x01, J12 Conn_01x01, J13 Conn_01x01, J14 Conn_01x01, J15 Conn_01x01, J16 Conn_01x01, J17 Conn_01x01, J18 Conn_01x01, J2 Conn_01x01, J22 Conn_01x09, J23 Conn_01x01, J3 Conn_01x01, J4 Conn_01x01, J5 Conn_01x01, J6 Conn_01x01, J7 Conn_01x01, J8 Conn_01x01, J9 Conn_01x01

Commit message: made the C3
Parts:
- removed J10, J11, J12, J13, J14, J15, J16, J17, J18, J2, J23, J3, J4, J5, J6, J7, J8, J9: Conn_01x01, FlexyPin:FlexyPin_1x01, symbol Connector_Generic:Conn_01x01
- added C1, C2: 1µF, Capacitor_SMD:C_0402_1005Metric, symbol Device:C_Small
- added D1: D, Diode_SMD:D_SOD-323, symbol Device:D_Small
- added J19: USB_C_Receptacle_USB2.0_14P, Connector_USB:USB_C_Receptacle_G-Switch_GT-USB-7010ASV, symbol Connector:USB_C_Receptacle_USB2.0_14P
- added J2, J3: Conn_01x09, flexypin:FlexyPin_1x09_P1.50mm, symbol Connector_Generic:Conn_01x09
- added R1, R2: 5,1kΩ, Resistor_SMD:R_0402_1005Metric, symbol Device:R_Small
- added R3: 10kΩ, Resistor_SMD:R_0402_1005Metric, symbol Device:R_Small
- added SW1, SW3: SW_Push, Button_Switch_SMD:SW_Push_SPST_NO_Alps_SKRK, symbol Switch:SW_Push
- added U1: RT9080, Package_TO_SOT_SMD:SOT-23-5, symbol Regulator_Linear:TLV75533PDBV
Connections:
- net EN: now also J2.2 (Pin_2), R3.2, SW3.1
- net GND: now also C1.1, C2.1, J19.A1 (GND), J19.A12 (GND), J19.B1 (GND), J19.B12 (GND), J19.S1 (SHIELD), J2.9 (Pin_9), R1.2, R2.2, SW1.2, SW3.2, U1.2 (GND)
- net IO0: now also J3.9 (Pin_9)
- net IO1: now also J3.8 (Pin_8)
- net IO10: now also J3.1 (Pin_1)
- net IO18: now also J19.A7 (D-), J19.B7 (D-), J3.4 (Pin_4)
- net IO19: now also J19.A6 (D+), J19.B6 (D+), J3.5 (Pin_5)
- net IO2: now also J3.7 (Pin_7)
- net IO3: now also J3.6 (Pin_6)
- net IO4: now also J2.3 (Pin_3)
- net IO5: now also J2.4 (Pin_4)
- net IO6: now also J2.5 (Pin_5)
- net IO7: now also J2.6 (Pin_6)
- net IO8: now also J2.7 (Pin_7)
- net IO9: now also J2.8 (Pin_8), SW1.1
- net RXD: now also J3.2 (Pin_2)
- net TXD: now also J3.3 (Pin_3)
- net 3.3V renamed +3.3V
- net +3.3V: now also C2.2, J2.1 (Pin_1), R3.1, U1.5 (OUT)
- new net: C1.2, D1.1 (K), U1.1 (IN), U1.3 (EN)
- new net: J19.A5 (CC1), R2.1
- new net: J19.B5 (CC2), R1.1
- new net +5V: D1.2 (A), J19.A4 (VBUS), J19.A9 (VBUS), J19.B4 (VBUS), J19.B9 (VBUS)
Other:
- moved on the sheet: J1, J22
