File: ESP32-S2_S3-WROOM_flexypin.kicad_pcb (KiCad board)
At the start: 2 copper layers, 31 x 51.4 mm, 28 parts, among them J1 Conn_01x20, J10 Conn_01x02, J11 Conn_01x02, J12 Conn_01x01, J13 Conn_01x02, J14 Conn_01x02, J15 Conn_01x02, J16 Conn_01x02, J17 Conn_01x02, J18 Conn_01x02, J19 Conn_01x02, J2 Conn_01x02, J20 Conn_01x02, J21 Conn_01x02, J22 Conn_01x20, J23 Conn_01x01, J3 Conn_01x02, J4 Conn_01x02, J5 Conn_01x02, J6 Conn_01x02, J7 Conn_01x02, J8 Conn_01x02, J9 Conn_01x02

Commit message: schematic etc
Parts:
- removed G*** (x2): LOGO, LOGO
- removed G*** (x2): LOGO, Symbols_Extra:SolderParty-New-Logo_10x8.5mm_SilkScreen
- removed J10, J11, J13, J14, J15, J16, J17, J18, J19, J20, J21, J3, J4, J5, J6, J7, J8, J9: Conn_01x02, FlexyPin:FlexyPin_1x02_P1.27mm
- removed J12, J23: Conn_01x01, FlexyPin:FlexyPin_1x01
- removed REF**: Fiducial_0.5mm_Mask1.5mm, Fiducial:Fiducial_0.5mm_Mask1.5mm
- added C1: 1µF, Capacitor_SMD:C_0402_1005Metric, F.Cu at (153.0, 118.9)
- added C2: 1µF, Capacitor_SMD:C_0402_1005Metric, F.Cu at (154.9, 118.9)
- added D1: D, Diode_SMD:D_SOD-323, F.Cu at (151.0, 121.5)
- added J24: USB_C_Receptacle_USB2.0_14P, Connector_USB:USB_C_Receptacle_G-Switch_GT-USB-7010ASV, F.Cu at (148.1, 128.8)
- added J25: Conn_01x12, flexypin:FlexyPin_1x12_P1.27mm, F.Cu at (141.1, 101.3)
- added J26: Conn_01x14, flexypin:FlexyPin_1x14_P1.27mm, F.Cu at (137.1, 81.3)
- added R1: 10kΩ, Resistor_SMD:R_0402_1005Metric, F.Cu at (141.0, 124.2)
- added R2: 5,1kΩ, Resistor_SMD:R_0402_1005Metric, F.Cu at (149.5, 122.8)
- added R3: 5,1kΩ, Resistor_SMD:R_0402_1005Metric, F.Cu at (145.5, 123.3)
- added SW1: SW_Push, Button_Switch_SMD:SW_Push_SPST_NO_Alps_SKRK, F.Cu at (141.0, 127.9)
- added SW2: SW_Push, Button_Switch_SMD:SW_Push_SPST_NO_Alps_SKRK, F.Cu at (155.1, 127.9)
- added U1: RT9080, Package_TO_SOT_SMD:SOT-23-5, F.Cu at (154.0, 121.5)
- J2: value Conn_01x02 -> Conn_01x14; footprint FlexyPin:FlexyPin_1x02_P1.27mm -> flexypin:FlexyPin_1x14_P1.27mm
- moved J2 27.6 mm to (159.1, 97.8), turned to 180 degrees
Connections:
- J1 pad 1: /GND -> GND
- J1 pad 13: /IO19 -> IO19
- J1 pad 14: /IO20 -> IO20
- J1 pad 2: /3.3V -> +3.3V
- J1 pad 3: /EN -> EN
- J2 pad 1: /GND -> IO0
- J2 pad 2: /3.3V -> /IO35
- J22 pad 1: /GND -> GND
- J22 pad 14: /IO0 -> IO0
Routing:
- net IO19: track 0.00 -> 54.7 mm, vias 0 -> 2
- net IO20: track 0.00 -> 50.0 mm, vias 0 -> 2
- net EN: track 0.00 -> 48.9 mm, vias 0 -> 1
- net IO0: track 0.00 -> 32.1 mm, vias 0 -> 1
- net GND: track 0.00 -> 28.9 mm
- net /GND: track 28.9 -> 0.00 mm
- net /IO19: track 20.9 -> 0.00 mm
- net /IO20: track 18.2 -> 0.00 mm
- net /IO0: track 18.2 -> 0.00 mm
- net +5V: track 0.00 -> 9.81 mm
- net Net-(D1-K): track 0.00 -> 6.81 mm
- net +3.3V: track 0.00 -> 6.37 mm, vias 0 -> 2
- net /EN: track 5.00 -> 0.00 mm
- net /3.3V: track 3.66 -> 0.00 mm
- net Net-(J24-CC1): track 0.00 -> 2.14 mm
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- added copper zone on B.Cu, net +3.3V
- added copper zone on F.Cu, net GND
Other:
- board text added: "GND IO1 IO2 TXD0 RXD0 IO42 IO41 IO40 IO39 IO38 IO37 IO36 IO35 IO0 IO45 IO34 IO47 IO48 IO14 IO13"
- board text removed: "ESP32-S2-SOLO ESP32-S3-WROOM Adapter Jan 2022"
- board text removed: "Module on this side"
