File: ESP32-S2_S3-WROOM_flexypin.kicad_sch (KiCad schematic)
At the start: 23 parts, among them J1 Conn_01x20, J10 Conn_01x02, J11 Conn_01x02, J12 Conn_01x01, J13 Conn_01x02, J14 Conn_01x02, J15 Conn_01x02, J16 Conn_01x02, J17 Conn_01x02, J18 Conn_01x02, J19 Conn_01x02, J2 Conn_01x02, J20 Conn_01x02, J21 Conn_01x02, J22 Conn_01x20, J23 Conn_01x01, J3 Conn_01x02, J4 Conn_01x02, J5 Conn_01x02, J6 Conn_01x02, J7 Conn_01x02, J8 Conn_01x02, J9 Conn_01x02

Commit message: schematic etc
Parts:
- removed J10, J11, J13, J14, J15, J16, J17, J18, J19, J2, J20, J21, J3, J4, J5, J6, J7, J8, J9: Conn_01x02, FlexyPin:FlexyPin_1x02_P1.27mm, symbol Connector_Generic:Conn_01x02
- removed J12, J23: Conn_01x01, FlexyPin:FlexyPin_1x01, symbol Connector_Generic:Conn_01x01
- added C1, C2: 1µF, Capacitor_SMD:C_0402_1005Metric, symbol Device:C_Small
- added D1: D, Diode_SMD:D_SOD-323, symbol Device:D_Small
- added J2, J26: Conn_01x14, flexypin:FlexyPin_1x14_P1.27mm, symbol Connector_Generic:Conn_01x14
- added J24: USB_C_Receptacle_USB2.0_14P, Connector_USB:USB_C_Receptacle_G-Switch_GT-USB-7010ASV, symbol Connector:USB_C_Receptacle_USB2.0_14P
- added J25: Conn_01x12, flexypin:FlexyPin_1x12_P1.27mm, symbol Connector_Generic:Conn_01x12
- added R1: 10kΩ, Resistor_SMD:R_0402_1005Metric, symbol Device:R_Small
- added R2, R3: 5,1kΩ, Resistor_SMD:R_0402_1005Metric, symbol Device:R_Small
- added SW1, SW2: SW_Push, Button_Switch_SMD:SW_Push_SPST_NO_Alps_SKRK, symbol Switch:SW_Push
- added U1: RT9080, Package_TO_SOT_SMD:SOT-23-5, symbol Regulator_Linear:TLV75533PDBV
Connections:
- net EN: now also J26.3 (Pin_3), R1.2, SW1.1
- net GND: now also C1.1, C2.1, J2.14 (Pin_14), J24.A1 (GND), J24.A12 (GND), J24.B1 (GND), J24.B12 (GND), J24.S1 (SHIELD), J26.1 (Pin_1), R2.2, R3.2, SW1.2, SW2.2, U1.2 (GND)
- net IO0: now also J2.1 (Pin_1), SW2.1
- net IO1: now also J2.13 (Pin_13)
- net IO10: now also J25.4 (Pin_4)
- net IO11: now also J25.5 (Pin_5)
- net IO12: now also J25.6 (Pin_6)
- net IO13: now also J25.7 (Pin_7)
- net IO14: now also J25.8 (Pin_8)
- net IO15: now also J26.8 (Pin_8)
- net IO16: now also J26.9 (Pin_9)
- net IO17: now also J26.10 (Pin_10)
- net IO18: now also J26.11 (Pin_11)
- net IO19: now also J24.A7 (D-), J24.B7 (D-), J26.13 (Pin_13)
- net IO2: now also J2.12 (Pin_12)
- net IO20: now also J24.A6 (D+), J24.B6 (D+), J26.14 (Pin_14)
- net IO21: now also J25.9 (Pin_9)
- net IO3: now also J25.1 (Pin_1)
- net IO33: now also J25.10 (Pin_10)
- net IO34: now also J25.11 (Pin_11)
- net IO35: now also J2.2 (Pin_2)
- net IO36: now also J2.3 (Pin_3)
- net IO37: now also J2.4 (Pin_4)
- net IO38: now also J2.5 (Pin_5)
- net IO39: now also J2.6 (Pin_6)
- net IO4: now also J26.4 (Pin_4)
- net IO40: now also J2.7 (Pin_7)
- net IO41: now also J2.8 (Pin_8)
- net IO42: now also J2.9 (Pin_9)
- net IO45: now also J25.12 (Pin_12)
- net IO46: now also J25.2 (Pin_2)
- net IO5: now also J26.5 (Pin_5)
- net IO6: now also J26.6 (Pin_6)
- net IO7: now also J26.7 (Pin_7)
- net IO8: now also J26.12 (Pin_12)
- net IO9: now also J25.3 (Pin_3)
- net RXD0: now also J2.10 (Pin_10)
- net TXD0: now also J2.11 (Pin_11)
- net 3.3V renamed +3.3V
- net +3.3V: now also C2.2, J26.2 (Pin_2), R1.1, U1.5 (OUT)
- new net: J24.B5 (CC2), R2.1
- new net: C1.2, D1.1 (K), U1.1 (IN), U1.3 (EN)
- new net: J24.A5 (CC1), R3.1
- new net +5V: D1.2 (A), J24.A4 (VBUS), J24.A9 (VBUS), J24.B4 (VBUS), J24.B9 (VBUS)
