File: ESP32-S2_S3-WROOM_flexypin.kicad_sch (KiCad schematic)
At the start: 15 parts, among them J1 Conn_01x20, J2 Conn_01x14, J22 Conn_01x20, J24 USB_C_Receptacle_USB2.0_14P, J25 Conn_01x12, J26 Conn_01x14, SW1 SW_Push, SW2 SW_Push, U1 RT9080

Commit message: mislabeling
Parts:
- added D2: LED_Small, LED_SMD:LED_0402_1005Metric, symbol Device:LED_Small
- added R4: 100-1kΩ, Resistor_SMD:R_0402_1005Metric, symbol Device:R_Small
Connections:
- net GND: now also R4.1
- net IO12: now also D2.2 (A)
- new net: D2.1 (K), R4.2
